Commit message: Imported upstream version '0.2.0' of 'upstream'

File: pincher_arm_description/urdf/arm_hardware.xacro (robot description, xacro)
@@ -1,4 +1,29 @@
 <?xml version="1.0"?>
-<!-- Basic URDF components for PhantomX Pincher Arm-->
+<!-- Basic URDF components for PhantomX Pincher Arm
+BSD 3-Clause License
+Copyright (c) 2021, Willow Garage, Inc.
+All rights reserved.
+Redistribution and use in source and binary forms, with or without
+modification, are permitted provided that the following conditions are met:
+    * Redistributions of source code must retain the above copyright
+      notice, this list of conditions and the following disclaimer.
+    * Redistributions in binary form must reproduce the above copyright
+      notice, this list of conditions and the following disclaimer in the
+      documentation and/or other materials provided with the distribution.
+    * Neither the name of the Willow Garage, Inc. nor the names of its
+      contributors may be used to endorse or promote products derived from
+      this software without specific prior written permission.
+THIS SOFTWARE IS PROVIDED BY THE COPYRIGHT HOLDERS AND CONTRIBUTORS "AS IS"
+AND ANY EXPRESS OR IMPLIED WARRANTIES, INCLUDING, BUT NOT LIMITED TO, THE
+IMPLIED WARRANTIES OF MERCHANTABILITY AND FITNESS FOR A PARTICULAR PURPOSE
+ARE DISCLAIMED. IN NO EVENT SHALL THE COPYRIGHT OWNER OR CONTRIBUTORS BE
+LIABLE FOR ANY DIRECT, INDIRECT, INCIDENTAL, SPECIAL, EXEMPLARY, OR
+CONSEQUENTIAL DAMAGES (INCLUDING, BUT NOT LIMITED TO, PROCUREMENT OF
+SUBSTITUTE GOODS OR SERVICES; LOSS OF USE, DATA, OR PROFITS; OR BUSINESS
+INTERRUPTION) HOWEVER CAUSED AND ON ANY THEORY OF LIABILITY, WHETHER IN
+CONTRACT, STRICT LIABILITY, OR TORT (INCLUDING NEGLIGENCE OR OTHERWISE)
+ARISING IN ANY WAY OUT OF THE USE OF THIS SOFTWARE, EVEN IF ADVISED OF THE
+POSSIBILITY OF SUCH DAMAGE.
+-->
 <robot xmlns:xacro="http://ros.org/wiki/xacro">
   <xacro:property name="M_SCALE" value="0.001"/>

File: pincher_arm_description/urdf/pincher_arm.urdf.xacro (robot description, xacro)
@@ -2,7 +2,4 @@
 <robot name="pincher_arm" xmlns:xacro="http://ros.org/wiki/xacro">
   <xacro:include filename="$(find pincher_arm_description)/urdf/pincher_arm.xacro"/>
-  <link name="base_link"/>
-  <xacro:pincher_arm parent="base_link">
-    <origin xyz="0.0 0.0 0.0"/>
-  </xacro:pincher_arm>
+  <xacro:pincher_arm/>
 </robot>

File: pincher_arm_description/urdf/pincher_arm.xacro (robot description, xacro)
@@ -1,4 +1,30 @@
 <?xml version="1.0"?>
-<!-- PhantomX Pincher arm description -->
+<!-- PhantomX Pincher arm description
+BSD 3-Clause License
+Copyright (c) 2021, Willow Garage, Inc.
+Copyright (c) 2021, Kell Ideas Ltd.
+All rights reserved.
+Redistribution and use in source and binary forms, with or without
+modification, are permitted provided that the following conditions are met:
+    * Redistributions of source code must retain the above copyright
+      notice, this list of conditions and the following disclaimer.
+    * Redistributions in binary form must reproduce the above copyright
+      notice, this list of conditions and the following disclaimer in the
+      documentation and/or other materials provided with the distribution.
+    * Neither the name of the Willow Garage, Inc. nor the names of its
+      contributors may be used to endorse or promote products derived from
+      this software without specific prior written permission.
+THIS SOFTWARE IS PROVIDED BY THE COPYRIGHT HOLDERS AND CONTRIBUTORS "AS IS"
+AND ANY EXPRESS OR IMPLIED WARRANTIES, INCLUDING, BUT NOT LIMITED TO, THE
+IMPLIED WARRANTIES OF MERCHANTABILITY AND FITNESS FOR A PARTICULAR PURPOSE
+ARE DISCLAIMED. IN NO EVENT SHALL THE COPYRIGHT OWNER OR CONTRIBUTORS BE
+LIABLE FOR ANY DIRECT, INDIRECT, INCIDENTAL, SPECIAL, EXEMPLARY, OR
+CONSEQUENTIAL DAMAGES (INCLUDING, BUT NOT LIMITED TO, PROCUREMENT OF
+SUBSTITUTE GOODS OR SERVICES; LOSS OF USE, DATA, OR PROFITS; OR BUSINESS
+INTERRUPTION) HOWEVER CAUSED AND ON ANY THEORY OF LIABILITY, WHETHER IN
+CONTRACT, STRICT LIABILITY, OR TORT (INCLUDING NEGLIGENCE OR OTHERWISE)
+ARISING IN ANY WAY OUT OF THE USE OF THIS SOFTWARE, EVEN IF ADVISED OF THE
+POSSIBILITY OF SUCH DAMAGE.
+-->
 <robot xmlns:xacro="http://ros.org/wiki/xacro">
   <xacro:include filename="$(find pincher_arm_description)/urdf/arm_hardware.xacro"/>
@@ -16,5 +42,4 @@
   </material>
   <xacro:macro name="pincher_arm" params="
-      parent:=base_link
       color:=Gray
       joints_vlimit:=1.571
@@ -28,12 +53,6 @@
       wrist_ulimit:=1.79
       gripper_llimit:=-2.6
-      gripper_ulimit:=0.0
-      *origin">
+      gripper_ulimit:=0.0">
     <link name="arm_base_link"/>
-    <joint name="arm_base_joint" type="fixed">
-      <xacro:insert_block name="origin"/>
-      <parent link="${parent}"/>
-      <child link="arm_base_link"/>
-    </joint>
     <!-- shoulder pan joint -->
     <xacro:dynamixel_AX12_fixed parent="arm_base_link" name="arm_shoulder_pan_servo">
